Commit message: feat: audit and resolve assembly system bugs; update configuration paths
- Fix TransformListener threading in assembly FSM with spin_thread=True
- Add missing part frame setup for main_bearing and small_bearing in state machine
- Correct ParameterValue type hints for boolean launch parameters across assembly cell
- Implement thread-safe force-torque capture with dedicated lock mechanism
- Add thread pool bounds to screwdriver server and grasp attacher for resource safety
- Improve spawn timing and FSM start delay for consistent part placement and vision readiness
- Add builtin_interfaces mock to FSM tests and update test suite to 38 passed
- Update MCP configuration path from /home/dark to /Users/darkdoll for cross-platform support
- Add comprehensive audit revision table to BUG_REPORT documenting status of all 37 reported issues
- Mark legacy URDF files and unused world configurations for deprecation
- Various configuration refinements for three-arm assembly cell bridging and sensor initialization

File: src/gearbox_sim/urdf/gearbox_gazebo.urdf.xacro (robot description, xacro)
@@ -90,7 +90,7 @@
   <xacro:macro name="sun_collision_mesh" params="">
     <collision>
-      <origin xyz="${-0.006872 * geom_factor} ${-0.006872 * geom_factor} ${-0.030400 * geom_factor}" rpy="0 0 0"/>
-      <geometry>
-        <mesh filename="file://$(find gearbox_sim)/meshes/satellite.STL" scale="${scale} ${scale} ${scale}"/>
+      <origin xyz="0 0 0" rpy="0 0 0"/>
+      <geometry>
+        <cylinder radius="${0.0070 * geom_factor}" length="${0.040 * geom_factor}"/>
       </geometry>
     </collision>
@@ -205,7 +205,7 @@
       <xacro:cylinder_inertia mass="${0.15 * mass_factor}" radius="${0.0070 * geom_factor}" length="${0.040 * geom_factor}"/>
       <visual>
-        <origin xyz="${-0.006872 * geom_factor} ${-0.006872 * geom_factor} ${-0.030400 * geom_factor}" rpy="0 0 0"/>
-        <geometry>
-          <mesh filename="file://$(find gearbox_sim)/meshes/satellite.STL" scale="${scale} ${scale} ${scale}"/>
+        <origin xyz="0 0 0" rpy="0 0 0"/>
+        <geometry>
+          <cylinder radius="${0.0070 * geom_factor}" length="${0.040 * geom_factor}"/>
         </geometry>
         <material name="blue"/>

File: src/gearbox_sim/urdf/include/workcell_macros.xacro (robot description, xacro)
@@ -553,4 +553,16 @@
       <dynamics damping="40.0" friction="6.0"/>
     </joint>
+    <gazebo reference="${prefix}ram_joint">
+      <sensor name="${prefix}ram_force_torque" type="force_torque">
+        <update_rate>250.0</update_rate>
+        <always_on>true</always_on>
+        <visualize>false</visualize>
+        <topic>/press/ft_sensor</topic>
+        <force_torque>
+          <frame>child</frame>
+          <measure_direction>parent_to_child</measure_direction>
+        </force_torque>
+      </sensor>
+    </gazebo>
     <!-- Frames -->
     <!-- bed_frame: where robot places parts — fixed at xyz[2]+0.13 (bolster top
